Commit message: add open_manipulator

File: src/youfork_description/urdf/youfork.urdf (robot description, URDF)
Before this commit: robot youfork, 11 links, 10 joints
Links:
- added link camera_link
- added link end_effector_link, mass 1.0e-03; visual box size=0.01 0.01 0.01
- added link gripper_link, mass 1.0e-03; collision mesh filename=package://open_manipulator_x_description/meshes/chain_link_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 scale=0.001 0.001 0.001; visual mesh filename=package://open_manipulator_x_description/meshes/chain_link_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 scale=0.001 0.001 0.001
- added link gripper_link_sub, mass 1.0e-03; collision mesh filename=package://open_manipulator_x_description/meshes/chain_link_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 scale=0.001 0.001 0.001; visual mesh filename=package://open_manipulator_x_description/meshes/chain_link_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 scale=0.001 0.001 0.001
- added link link1, mass 7.9119962e-02; collision mesh filename=package://open_manipulator_x_description/meshes/chain_link1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 scale=0.001 0.001 0.001; visual mesh filename=package://open_manipulator_x_description/meshes/chain_link1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 scale=0.001 0.001 0.001
- added link link2, mass 9.8406837e-02; collision mesh filename=package://open_manipulator_x_description/meshes/chain_link2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 scale=0.001 0.001 0.001; visual mesh filename=package://open_manipulator_x_description/meshes/chain_link2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 scale=0.001 0.001 0.001
- added link link3, mass 1.3850917e-01; collision mesh filename=package://open_manipulator_x_description/meshes/chain_link3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 scale=0.001 0.001 0.001; visual mesh filename=package://open_manipulator_x_description/meshes/chain_link3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 scale=0.001 0.001 0.001
- added link link4, mass 1.3274562e-01; collision mesh filename=package://open_manipulator_x_description/meshes/chain_link4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 scale=0.001 0.001 0.001; visual mesh filename=package://open_manipulator_x_description/meshes/chain_link4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 scale=0.001 0.001 0.001
- added link link5, mass 1.4327573e-01; collision mesh filename=package://open_manipulator_x_description/meshes/chain_link5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 scale=0.001 0.001 0.001; visual mesh filename=package://open_manipulator_x_description/meshes/chain_link5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 scale=0.001 0.001 0.001
Joints:
- added joint camera_joint: type fixed, parent link5, child camera_link, origin xyz=0.070 0.032 0.052 rpy=0 0 0, axis 0 1 0
- added joint end_effector_joint: type fixed, parent link5, child end_effector_link, origin xyz=0.126 0.0 0.0 rpy=0 0 0
- added joint gripper: type prismatic, parent link5, child gripper_link, origin xyz=0.0817 0.021 0.0 rpy=0 0 0, axis 0 1 0, limit lower=-0.010 upper=0.019 effort=1 velocity=4.8
- added joint gripper_sub: type prismatic, parent link5, child gripper_link_sub, origin xyz=0.0817 -0.021 0.0 rpy=0 0 0, axis 0 -1 0, limit lower=-0.010 upper=0.019 effort=1 velocity=4.8, mimic joint=gripper multiplier=1
- added joint joint1: type revolute, parent link1, child link2, origin xyz=0.012 0.0 0.017 rpy=0 0 0, axis 0 0 1, limit lower=-2.82743338823 upper=2.82743338823 effort=1 velocity=4.8
- added joint joint2: type revolute, parent link2, child link3, origin xyz=0.0 0.0 0.0595 rpy=0 0 0, axis 0 1 0, limit lower=-1.79070781255 upper=1.57079632679 effort=1 velocity=4.8
- added joint joint3: type revolute, parent link3, child link4, origin xyz=0.024 0 0.128 rpy=0 0 0, axis 0 1 0, limit lower=-0.94247779607 upper=1.38230076758 effort=1 velocity=4.8
- added joint joint4: type revolute, parent link4, child link5, origin xyz=0.124 0.0 0.0 rpy=0 0 0, axis 0 1 0, limit lower=-1.79070781255 upper=2.04203522483 effort=1 velocity=4.8
- added joint origin_to_link1: type fixed, parent base_link, child link1, origin xyz=0 0 0 rpy=0 0 0, axis 0 0 1

File: src/youfork_description/urdf/youfork.urdf.xacro (robot description, xacro)
@@ -2,11 +2,11 @@
 <robot name="youfork" xmlns:xacro="http://ros.org/wiki/xacro">
   <xacro:include filename="$(find ca_description)/urdf/create_base.urdf.xacro" />
-  <!-- <xacro:include filename="$(find ca_description)/urdf/create_2_gazebo.urdf.xacro" /> -->
-  <!-- <xacro:include filename="$(find open_manipulator_x_description)/urdf/materials.xacro" /> -->
-  <!-- <xacro:include filename="$(find open_manipulator_x_description)/urdf/open_manipulator_x.gazebo.xacro" /> -->
-  <!-- <xacro:include filename="$(find open_manipulator_x_description)/urdf/open_manipulator_x.transmission.xacro" /> -->
-  <!-- <xacro:include filename="$(find open_manipulator_x_description)/urdf/open_manipulator_x.urdf.xacro" /> -->
+  <xacro:include filename="$(find ca_description)/urdf/create_2_gazebo.urdf.xacro" />
+  <xacro:include filename="$(find open_manipulator_x_description)/urdf/open_manipulator_x_robot.urdf.xacro" />
   <xacro:create_base wheel_separation="0.235" base_diameter="0.3485">
     <mesh filename="package://ca_description/meshes/create_2.dae" />
   </xacro:create_base>
+  <xacro:open_manipulator_x parent="base_link">
+    <origin xyz="0 0 0" rpy="0 0 0" />
+  </xacro:open_manipulator_x>
 </robot>

Commit message: fix correct position

File: src/youfork_description/urdf/youfork.urdf (robot description, URDF)
Before this commit: robot youfork, 20 links, 19 joints
Joints:
- joint origin_to_link1: origin xyz=0 0 0 rpy=0 0 0 -> xyz=0.1 0 0.1 rpy=0 -1.5708 0

File: src/youfork_description/urdf/youfork.urdf.xacro (robot description, xacro)
@@ -8,5 +8,5 @@
   </xacro:create_base>
   <xacro:open_manipulator_x parent="base_link">
-    <origin xyz="0 0 0" rpy="0 0 0" />
+    <origin xyz="0.1 0 0.1" rpy="0 -1.5708 0" />
   </xacro:open_manipulator_x>
 </robot>

Commit message: add battery and xavier

File: src/youfork_description/urdf/youfork.urdf (robot description, URDF)
Before this commit: robot youfork, 20 links, 19 joints
Links:
- added link jetson_xavier, mass 1.548; collision box size=0.105 0.105 0.065; visual box size=0.105 0.105 0.065
- added link krisdonia_battery, mass 0.680389; collision box size=0.127 0.14986 0.02794; visual box size=0.127 0.14986 0.02794
Joints:
- added joint jetson_xavier_to_base_link: type fixed, parent base_link, child jetson_xavier, origin xyz=-0.02 -0.09 0.11 rpy=0 0 0
- added joint krisdonia_battery_to_base_link: type fixed, parent base_link, child krisdonia_battery, origin xyz=0 0.1 0.09 rpy=0 0 1.5708

File: src/youfork_description/urdf/youfork.urdf.xacro (robot description, xacro)
@@ -10,3 +10,51 @@
     <origin xyz="0.1 0 0.1" rpy="0 -1.5708 0" />
   </xacro:open_manipulator_x>
+  <link name="jetson_xavier">
+    <inertial>
+      <origin xyz="0 0 0" rpy="0 0 0"/>
+      <mass value="1.548"/>
+      <inertia ixx="100"  ixy="0"  ixz="0" iyy="100" iyz="0" izz="100" />
+    </inertial>
+    <visual>
+      <origin xyz="0 0 0" rpy="0 0 0" />
+      <geometry>
+        <box size="0.105 0.105 0.065" />
+      </geometry>
+    </visual>
+    <collision>
+      <origin xyz="0 0 0" rpy="0 0 0" />
+      <geometry>
+        <box size="0.105 0.105 0.065" />
+      </geometry>
+    </collision>
+  </link>
+  <joint name="jetson_xavier_to_base_link" type="fixed">
+    <origin xyz="-0.02 -0.09 0.11" rpy="0 0 0"/>
+    <parent link="base_link"/>
+    <child link="jetson_xavier"/>
+  </joint>
+  <link name="krisdonia_battery">
+    <inertial>
+      <origin xyz="0 0 0" rpy="0 0 0"/>
+      <mass value="0.680389"/>
+      <inertia ixx="100"  ixy="0"  ixz="0" iyy="100" iyz="0" izz="100" />
+    </inertial>
+    <visual>
+      <origin xyz="0 0 0" rpy="0 0 0" />
+      <geometry>
+        <box size="0.127 0.14986 0.02794" />
+      </geometry>
+    </visual>
+    <collision>
+      <origin xyz="0 0 0" rpy="0 0 0" />
+      <geometry>
+        <box size="0.127 0.14986 0.02794" />
+      </geometry>
+    </collision>
+  </link>
+  <joint name="krisdonia_battery_to_base_link" type="fixed">
+    <origin xyz="0 0.1 0.09" rpy="0 0 1.5708"/>
+    <parent link="base_link"/>
+    <child link="krisdonia_battery"/>
+  </joint>
 </robot>

Commit message: add d435

File: src/youfork_description/urdf/youfork.urdf (robot description, URDF)
Before this commit: robot youfork, 22 links, 21 joints
Links:
- added link d435_bottom_screw_frame
- added link d435_color_frame
- added link d435_color_optical_frame
- added link d435_depth_frame
- added link d435_depth_optical_frame
- added link d435_infra1_frame
- added link d435_infra1_optical_frame
- added link d435_infra2_frame
- added link d435_infra2_optical_frame
- added link d435_link, mass 0.564; collision box size=0.02505 0.09 0.025; visual mesh filename=package://realsense2_description/meshes/d435.dae
Joints:
- added joint d435_color_joint: type fixed, parent d435_link, child d435_color_frame, origin xyz=0 0.015 0 rpy=0 0 0
- added joint d435_color_optical_joint: type fixed, parent d435_color_frame, child d435_color_optical_frame, origin xyz=0 0 0 rpy=-1.5707963267948966 0 -1.5707963267948966
- added joint d435_depth_joint: type fixed, parent d435_link, child d435_depth_frame, origin xyz=0 0 0 rpy=0 0 0
- added joint d435_depth_optical_joint: type fixed, parent d435_depth_frame, child d435_depth_optical_frame, origin xyz=0 0 0 rpy=-1.5707963267948966 0 -1.5707963267948966
- added joint d435_infra1_joint: type fixed, parent d435_link, child d435_infra1_frame, origin xyz=0 0.0 0 rpy=0 0 0
- added joint d435_infra1_optical_joint: type fixed, parent d435_infra1_frame, child d435_infra1_optical_frame, origin xyz=0 0 0 rpy=-1.5707963267948966 0 -1.5707963267948966
- added joint d435_infra2_joint: type fixed, parent d435_link, child d435_infra2_frame, origin xyz=0 -0.05 0 rpy=0 0 0
- added joint d435_infra2_optical_joint: type fixed, parent d435_infra2_frame, child d435_infra2_optical_frame, origin xyz=0 0 0 rpy=-1.5707963267948966 0 -1.5707963267948966
- added joint d435_joint: type fixed, parent base_link, child d435_bottom_screw_frame, origin xyz=0.12 0 0.09 rpy=0 -0.17453 0
- added joint d435_link_joint: type fixed, parent d435_bottom_screw_frame, child d435_link, origin xyz=0.010600000000000002 0.0175 0.0125 rpy=0 0 0

File: src/youfork_description/urdf/youfork.urdf.xacro (robot description, xacro)
@@ -4,4 +4,5 @@
   <xacro:include filename="$(find ca_description)/urdf/create_2_gazebo.urdf.xacro" />
   <xacro:include filename="$(find open_manipulator_x_description)/urdf/open_manipulator_x_robot.urdf.xacro" />
+  <xacro:include filename="$(find realsense2_description)/urdf/_d435.urdf.xacro" />
   <xacro:create_base wheel_separation="0.235" base_diameter="0.3485">
     <mesh filename="package://ca_description/meshes/create_2.dae" />
@@ -10,4 +11,7 @@
     <origin xyz="0.1 0 0.1" rpy="0 -1.5708 0" />
   </xacro:open_manipulator_x>
+  <xacro:sensor_d435 parent="base_link" name="d435">
+    <origin xyz="0.12 0 0.08" rpy="0 -0.17453 0"/>
+  </xacro:sensor_d435>
   <link name="jetson_xavier">
     <inertial>

Commit message: add rplidar but too big

File: src/youfork_description/urdf/youfork.urdf (robot description, URDF)
Before this commit: robot youfork, 32 links, 31 joints
Links:
- added link rplidar, mass 0.190; collision mesh filename=package://youfork_description/meshes/rplidar_main.STL; visual mesh filename=package://youfork_description/meshes/rplidar_main.STL
Joints:
- added joint rplidar_to_base_link: type fixed, parent base_link, child rplidar, origin xyz=0.2 0.0 0.1 rpy=0 0 0
- joint d435_joint: origin xyz=0.12 0 0.09 rpy=0 -0.17453 0 -> xyz=0.12 0 0.08 rpy=0 -0.17453 0

File: src/youfork_description/urdf/youfork.urdf.xacro (robot description, xacro)
@@ -14,4 +14,28 @@
     <origin xyz="0.12 0 0.08" rpy="0 -0.17453 0"/>
   </xacro:sensor_d435>
+  <link name="rplidar">
+    <inertial>
+      <origin xyz="0 0 0" rpy="0 0 0"/>
+      <mass value="0.190"/>
+      <inertia ixx="100"  ixy="0"  ixz="0" iyy="100" iyz="0" izz="100" />
+    </inertial>
+    <visual>
+      <origin xyz="0 0 0" rpy="0 0 0" />
+      <geometry>
+        <mesh filename="package://youfork_description/meshes/rplidar_main.STL" />
+      </geometry>
+    </visual>
+    <collision>
+      <origin xyz="0 0 0" rpy="0 0 0" />
+      <geometry>
+        <mesh filename="package://youfork_description/meshes/rplidar_main.STL" />
+      </geometry>
+    </collision>
+  </link>
+  <joint name="rplidar_to_base_link" type="fixed">
+    <origin xyz="0.2 0.0 0.1" rpy="0 0 0"/>
+    <parent link="base_link"/>
+    <child link="rplidar"/>
+  </joint>
   <link name="jetson_xavier">
     <inertial>

Commit message: fix rplidar location

File: src/youfork_description/urdf/youfork.urdf (robot description, URDF)
Before this commit: robot youfork, 33 links, 32 joints
Links:
- link rplidar: geometry collision mesh filename=package://youfork_description/meshes/rplidar_main.STL scale=0.001 0.001 0.001; visual mesh filename=package://youfork_description/meshes/rplidar_main.STL scale=0.001 0.001 0.001
Joints:
- removed joint rplidar_to_base_link
- added joint rplidar_to_camera_link: type fixed, parent camera_link, child rplidar, origin xyz=0 0 0 rpy=0 0 0

File: src/youfork_description/urdf/youfork.urdf.xacro (robot description, xacro)
@@ -21,19 +21,19 @@
     </inertial>
     <visual>
-      <origin xyz="0 0 0" rpy="0 0 0" />
+      <origin xyz="0 -0.035 0" rpy="1.570796 0 3.14159" />
       <geometry>
-        <mesh filename="package://youfork_description/meshes/rplidar_main.STL" />
+        <mesh filename="package://youfork_description/meshes/rplidar_main.STL" scale="0.001 0.001 0.001" />
       </geometry>
     </visual>
     <collision>
-      <origin xyz="0 0 0" rpy="0 0 0" />
+      <origin xyz="0 -0.035 0" rpy="1.570796 0 3.14159" />
       <geometry>
-        <mesh filename="package://youfork_description/meshes/rplidar_main.STL" />
+        <mesh filename="package://youfork_description/meshes/rplidar_main.STL" scale="0.001 0.001 0.001" />
       </geometry>
     </collision>
   </link>
-  <joint name="rplidar_to_base_link" type="fixed">
-    <origin xyz="0.2 0.0 0.1" rpy="0 0 0"/>
-    <parent link="base_link"/>
+  <joint name="rplidar_to_camera_link" type="fixed">
+    <origin xyz="0 0 0" rpy="0 0 0"/>
+    <parent link="camera_link"/>
     <child link="rplidar"/>
   </joint>
